Commit message: Airplane work

File: crane_x7_description/urdf/crane_x7_arm.xacro (robot description, xacro)
@@ -4,5 +4,4 @@
   <xacro:property name="SCALE_MM" value="0.001"/>
   <xacro:property name="SCALE_CM" value="0.01"/>
-  <xacro:property name="BASE_FIXED_PART_HEIGHT" value="0.005"/>
   <!-- Macro for the standard CRANE X7 configuration -->
   <xacro:macro name="crane_x7_arm"
@@ -77,4 +76,17 @@
       <origin xyz="0 0 0" rpy="0 0 0"/>
     </crane_x7_wrist>
+    <!-- Export joint names using CRANE X7 default configuration part names -->
+    <xacro:property name="CRANE_X7_SHOULDER_PAN_JOINT_NAME"
+        value="${CRANE_X7_BASE_PAN_JOINT_NAME}"/>
+    <xacro:property name="CRANE_X7_SHOULDER_TILT_JOINT_NAME"
+        value="${CRANE_X7_BASE_TILT_JOINT_NAME}"/>
+    <xacro:property name="CRANE_X7_UPPER_ARM_TWIST_JOINT_NAME"
+        value="${CRANE_X7_ROTLINK_1_TWIST_JOINT_NAME}"/>
+    <xacro:property name="CRANE_X7_UPPER_ARM_ROTATE_JOINT_NAME"
+        value="${CRANE_X7_ROTLINK_1_ROTATE_JOINT_NAME}"/>
+    <xacro:property name="CRANE_X7_LOWER_ARM_TWIST_JOINT_NAME"
+        value="${CRANE_X7_ROTLINK_2_TWIST_JOINT_NAME}"/>
+    <xacro:property name="CRANE_X7_LOWER_ARM_ROTATE_JOINT_NAME"
+        value="${CRANE_X7_ROTLINK_2_ROTATE_JOINT_NAME}"/>
   </xacro:macro>
   <!-- Composite parts -->
@@ -187,5 +199,6 @@
     </link>
     <!-- Pan joint of the shoulder -->
-    <joint name="${name}_pan_joint" type="revolute">
+    <xacro:property name="CRANE_X7_BASE_PAN_JOINT_NAME" value="${name}_pan_joint"/>
+    <joint name="${CRANE_X7_BASE_PAN_JOINT_NAME}" type="revolute">
       <origin xyz="0 0 ${BASE_FIXED_PART_JOINT_Z}" rpy="0 0 0"/>
       <axis xyz="0 0 1"/>
@@ -224,5 +237,6 @@
     </link>
     <!-- Tilt joint of the shoulder -->
-    <joint name="${name}_tilt_joint" type="revolute">
+    <xacro:property name="CRANE_X7_BASE_TILT_JOINT_NAME" value="${name}_tilt_joint"/>
+    <joint name="${CRANE_X7_BASE_TILT_JOINT_NAME}" type="revolute">
       <origin xyz="0 0 ${BASE_REVOLUTE_PART_JOINT_Z}" rpy="0 0 0"/>
       <axis xyz="0 1 0"/>
@@ -327,5 +341,6 @@
         rotate_vlimit rotate_llimit rotate_ulimit attached_link">
     <!-- Joint for twisting around long axis -->
-    <joint name="${name}_twist_joint" type="revolute">
+    <xacro:property name="CRANE_X7_ROTLINK_1_TWIST_JOINT_NAME" value="${name}_twist_joint"/>
+    <joint name="${CRANE_X7_ROTLINK_1_TWIST_JOINT_NAME}" type="revolute">
       <origin xyz="0 0 ${TYPE_1_FIXED_PART_JOINT_Z}" rpy="0 0 0"/>
       <axis xyz="0 0 1"/>
@@ -362,5 +377,6 @@
     </link>
     <!-- Joint for rotating the attached part -->
-    <joint name="${name}_rotate_joint" type="revolute">
+    <xacro:property name="CRANE_X7_ROTLINK_1_ROTATE_JOINT_NAME" value="${name}_rotate_joint"/>
+    <joint name="${CRANE_X7_ROTLINK_1_ROTATE_JOINT_NAME}" type="revolute">
       <origin xyz="0 0 ${TYPE_1_REVOLUTE_PART_JOINT_Z}" rpy="0 0 0"/>
       <axis xyz="0 -1 0"/>
@@ -401,5 +417,6 @@
       </inertial>
     </link>
-    <joint name="${name}_joint" type="revolute">
+    <xacro:property name="CRANE_X7_ROTLINK_2_TWIST_JOINT_NAME" value="${name}_joint"/>
+    <joint name="${CRANE_X7_ROTLINK_2_TWIST_JOINT_NAME}" type="revolute">
       <origin xyz="0 0 ${TYPE_2_FIXED_PART_JOINT_Z}" rpy="0 0 0"/>
       <axis xyz="0 0 1"/>
@@ -497,5 +514,6 @@
       </inertial>
     </link>
-    <joint name="${name}_joint" type="revolute">
+    <xacro:property name="CRANE_X7_ROTLINK_2_ROTATE_JOINT_NAME" value="${name}_joint"/>
+    <joint name="${CRANE_X7_ROTLINK_2_ROTATE_JOINT_NAME}" type="revolute">
       <origin xyz="0 0 ${TYPE_2_REVOLUTE_PART_JOINT_Z}" rpy="0 0 0"/>
       <axis xyz="0 1 0"/>
@@ -537,5 +555,6 @@
       </inertial>
     </link>
-    <joint name="${name}_joint" type="revolute">
+    <xacro:property name="CRANE_X7_WRIST_JOINT_NAME" value="${name}_joint"/>
+    <joint name="${CRANE_X7_WRIST_JOINT_NAME}" type="revolute">
       <origin xyz="0 0 ${WRIST_JOINT_Z}" rpy="0 0 0"/>
       <axis xyz="0 0 1"/>

File: crane_x7_description/urdf/crane_x7_wide_two_finger_gripper.xacro (robot description, xacro)
@@ -30,5 +30,6 @@
       </inertial>
     </link>
-    <joint name="${name}_finger_a_joint" type="revolute">
+    <xacro:property name="CRANE_X7_WTFG_FINGER_A_JOINT_NAME" value="${name}_finger_a_joint"/>
+    <joint name="${CRANE_X7_WTFG_FINGER_A_JOINT_NAME}" type="revolute">
       <origin xyz="-0.012 0.0 0.024" rpy="0 0 0"/>
       <axis xyz="0 -1 0"/>
@@ -61,5 +62,6 @@
       </inertial>
     </link>
-    <joint name="${name}_finger_b_joint" type="revolute">
+    <xacro:property name="CRANE_X7_WTFG_FINGER_B_JOINT_NAME" value="${name}_finger_b_joint"/>
+    <joint name="${CRANE_X7_WTFG_FINGER_A_JOINT_NAME}" type="revolute">
       <origin xyz="0.012 0.0 0.024" rpy="0 0 0"/>
       <axis xyz="0 1 0"/>

Commit message: Fix non-global parameters for joint names

File: crane_x7_description/urdf/crane_x7_arm.xacro (robot description, xacro)
@@ -78,15 +78,21 @@
     <!-- Export joint names using CRANE X7 default configuration part names -->
     <xacro:property name="CRANE_X7_SHOULDER_PAN_JOINT_NAME"
-        value="${CRANE_X7_BASE_PAN_JOINT_NAME}"/>
+        value="${CRANE_X7_BASE_PAN_JOINT_NAME}"
+        scope="global"/>
     <xacro:property name="CRANE_X7_SHOULDER_TILT_JOINT_NAME"
-        value="${CRANE_X7_BASE_TILT_JOINT_NAME}"/>
+        value="${CRANE_X7_BASE_TILT_JOINT_NAME}"
+        scope="global"/>
     <xacro:property name="CRANE_X7_UPPER_ARM_TWIST_JOINT_NAME"
-        value="${CRANE_X7_ROTLINK_1_TWIST_JOINT_NAME}"/>
+        value="${CRANE_X7_ROTLINK_1_TWIST_JOINT_NAME}"
+        scope="global"/>
     <xacro:property name="CRANE_X7_UPPER_ARM_ROTATE_JOINT_NAME"
-        value="${CRANE_X7_ROTLINK_1_ROTATE_JOINT_NAME}"/>
+        value="${CRANE_X7_ROTLINK_1_ROTATE_JOINT_NAME}"
+        scope="global"/>
     <xacro:property name="CRANE_X7_LOWER_ARM_TWIST_JOINT_NAME"
-        value="${CRANE_X7_ROTLINK_2_TWIST_JOINT_NAME}"/>
+        value="${CRANE_X7_ROTLINK_2_TWIST_JOINT_NAME}"
+        scope="global"/>
     <xacro:property name="CRANE_X7_LOWER_ARM_ROTATE_JOINT_NAME"
-        value="${CRANE_X7_ROTLINK_2_ROTATE_JOINT_NAME}"/>
+        value="${CRANE_X7_ROTLINK_2_ROTATE_JOINT_NAME}"
+        scope="global"/>
   </xacro:macro>
   <!-- Composite parts -->
@@ -199,5 +205,5 @@
     </link>
     <!-- Pan joint of the shoulder -->
-    <xacro:property name="CRANE_X7_BASE_PAN_JOINT_NAME" value="${name}_pan_joint"/>
+    <xacro:property name="CRANE_X7_BASE_PAN_JOINT_NAME" value="${name}_pan_joint" scope="global"/>
     <joint name="${CRANE_X7_BASE_PAN_JOINT_NAME}" type="revolute">
       <origin xyz="0 0 ${BASE_FIXED_PART_JOINT_Z}" rpy="0 0 0"/>
@@ -237,5 +243,5 @@
     </link>
     <!-- Tilt joint of the shoulder -->
-    <xacro:property name="CRANE_X7_BASE_TILT_JOINT_NAME" value="${name}_tilt_joint"/>
+    <xacro:property name="CRANE_X7_BASE_TILT_JOINT_NAME" value="${name}_tilt_joint" scope="global"/>
     <joint name="${CRANE_X7_BASE_TILT_JOINT_NAME}" type="revolute">
       <origin xyz="0 0 ${BASE_REVOLUTE_PART_JOINT_Z}" rpy="0 0 0"/>
@@ -341,5 +347,5 @@
         rotate_vlimit rotate_llimit rotate_ulimit attached_link">
     <!-- Joint for twisting around long axis -->
-    <xacro:property name="CRANE_X7_ROTLINK_1_TWIST_JOINT_NAME" value="${name}_twist_joint"/>
+    <xacro:property name="CRANE_X7_ROTLINK_1_TWIST_JOINT_NAME" value="${name}_twist_joint" scope="global"/>
     <joint name="${CRANE_X7_ROTLINK_1_TWIST_JOINT_NAME}" type="revolute">
       <origin xyz="0 0 ${TYPE_1_FIXED_PART_JOINT_Z}" rpy="0 0 0"/>
@@ -377,5 +383,5 @@
     </link>
     <!-- Joint for rotating the attached part -->
-    <xacro:property name="CRANE_X7_ROTLINK_1_ROTATE_JOINT_NAME" value="${name}_rotate_joint"/>
+    <xacro:property name="CRANE_X7_ROTLINK_1_ROTATE_JOINT_NAME" value="${name}_rotate_joint" scope="global"/>
     <joint name="${CRANE_X7_ROTLINK_1_ROTATE_JOINT_NAME}" type="revolute">
       <origin xyz="0 0 ${TYPE_1_REVOLUTE_PART_JOINT_Z}" rpy="0 0 0"/>
@@ -417,5 +423,5 @@
       </inertial>
     </link>
-    <xacro:property name="CRANE_X7_ROTLINK_2_TWIST_JOINT_NAME" value="${name}_joint"/>
+    <xacro:property name="CRANE_X7_ROTLINK_2_TWIST_JOINT_NAME" value="${name}_joint" scope="global"/>
     <joint name="${CRANE_X7_ROTLINK_2_TWIST_JOINT_NAME}" type="revolute">
       <origin xyz="0 0 ${TYPE_2_FIXED_PART_JOINT_Z}" rpy="0 0 0"/>
@@ -514,5 +520,5 @@
       </inertial>
     </link>
-    <xacro:property name="CRANE_X7_ROTLINK_2_ROTATE_JOINT_NAME" value="${name}_joint"/>
+    <xacro:property name="CRANE_X7_ROTLINK_2_ROTATE_JOINT_NAME" value="${name}_joint" scope="global"/>
     <joint name="${CRANE_X7_ROTLINK_2_ROTATE_JOINT_NAME}" type="revolute">
       <origin xyz="0 0 ${TYPE_2_REVOLUTE_PART_JOINT_Z}" rpy="0 0 0"/>
@@ -555,5 +561,5 @@
       </inertial>
     </link>
-    <xacro:property name="CRANE_X7_WRIST_JOINT_NAME" value="${name}_joint"/>
+    <xacro:property name="CRANE_X7_WRIST_JOINT_NAME" value="${name}_joint" scope="global"/>
     <joint name="${CRANE_X7_WRIST_JOINT_NAME}" type="revolute">
       <origin xyz="0 0 ${WRIST_JOINT_Z}" rpy="0 0 0"/>

File: crane_x7_description/urdf/crane_x7_wide_two_finger_gripper.xacro (robot description, xacro)
@@ -30,5 +30,7 @@
       </inertial>
     </link>
-    <xacro:property name="CRANE_X7_WTFG_FINGER_A_JOINT_NAME" value="${name}_finger_a_joint"/>
+    <xacro:property name="CRANE_X7_WTFG_FINGER_A_JOINT_NAME"
+      value="${name}_finger_a_joint"
+      scope="global"/>
     <joint name="${CRANE_X7_WTFG_FINGER_A_JOINT_NAME}" type="revolute">
       <origin xyz="-0.012 0.0 0.024" rpy="0 0 0"/>
@@ -62,6 +64,8 @@
       </inertial>
     </link>
-    <xacro:property name="CRANE_X7_WTFG_FINGER_B_JOINT_NAME" value="${name}_finger_b_joint"/>
-    <joint name="${CRANE_X7_WTFG_FINGER_A_JOINT_NAME}" type="revolute">
+    <xacro:property name="CRANE_X7_WTFG_FINGER_B_JOINT_NAME"
+      value="${name}_finger_b_joint"
+      scope="global"/>
+    <joint name="${CRANE_X7_WTFG_FINGER_B_JOINT_NAME}" type="revolute">
       <origin xyz="0.012 0.0 0.024" rpy="0 0 0"/>
       <axis xyz="0 1 0"/>

File: crane_x7_simulation/urdf/crane_x7_transmissions.xacro (robot description, xacro)
@@ -71,5 +71,5 @@
   </xacro:macro>
   <!-- Generic transmission for use by joints that are not unique -->
-  <xacro:macro name="crane_x7_generic_transmissions" params="joint_name">
+  <xacro:macro name="crane_x7_generic_transmission" params="joint_name">
     <transmission name="${joint_name}_transmission">
       <type>transmission_interface/SimpleTransmission</type>

File: crane_x7_simulation/urdf/simulated_crane_x7.sdf.xacro (robot description, xacro)
@@ -48,13 +48,13 @@
     <plugin name="joint_state_publisher" filename="libgazebo_ros_joint_state_publisher.so">
       <jointName>
-        ${CRANE_X7_SHOULDER_PAN_JOINT_NAME,
-        ${CRANE_X7_SHOULDER_TILT_JOINT_NAME,
-        ${CRANE_X7_UPPER_ARM_TWIST_JOINT_NAME,
-        ${CRANE_X7_UPPER_ARM_ROTATE_JOINT_NAME,
-        ${CRANE_X7_LOWER_ARM_TWIST_JOINT_NAME,
-        ${CRANE_X7_LOWER_ARM_ROTATE_JOINT_NAME,
-        ${CRANE_X7_WRIST_JOINT_NAME,
-        ${CRANE_X7_WTFG_FINGER_A_JOINT_NAME,
-        ${CRANE_X7_WTFG_FINGER_B_JOINT_NAME,
+        ${CRANE_X7_SHOULDER_PAN_JOINT_NAME},
+        ${CRANE_X7_SHOULDER_TILT_JOINT_NAME},
+        ${CRANE_X7_UPPER_ARM_TWIST_JOINT_NAME},
+        ${CRANE_X7_UPPER_ARM_ROTATE_JOINT_NAME},
+        ${CRANE_X7_LOWER_ARM_TWIST_JOINT_NAME},
+        ${CRANE_X7_LOWER_ARM_ROTATE_JOINT_NAME},
+        ${CRANE_X7_WRIST_JOINT_NAME},
+        ${CRANE_X7_WTFG_FINGER_A_JOINT_NAME},
+        ${CRANE_X7_WTFG_FINGER_B_JOINT_NAME},
       </jointName>
     </plugin>
